Commit message: testing Diffbot with Gazebo

File: description/ros2_control/diffbot.ros2_control.xacro (robot description, xacro)
@@ -1,5 +1,5 @@
 <?xml version="1.0"?>
 <robot xmlns:xacro="http://www.ros.org/wiki/xacro">
-  <xacro:macro name="diffbot_ros2_control" params="name prefix use_mock_hardware">
+  <xacro:macro name="diffbot_ros2_control" params="name prefix use_mock_hardware use_gazebo_classic">
     <ros2_control name="${name}" type="system">
       <xacro:unless value="${use_mock_hardware}">
@@ -16,4 +16,9 @@
         </hardware>
       </xacro:if>
+      <xacro:if value="${use_gazebo_classic}">
+          <hardware>
+              <plugin>gazebo_ros2_control/GazeboSystem</plugin>
+          </hardware>
+      </xacro:if>
       <joint name="${prefix}left_wheel_joint">
         <command_interface name="velocity"/>

File: description/urdf/diffbot.urdf.xacro (robot description, xacro)
@@ -4,4 +4,5 @@
   <xacro:arg name="prefix" default="" />
   <xacro:arg name="use_mock_hardware" default="false" />
+  <xacro:arg name="use_gazebo_classic" default="false" />
   <xacro:include filename="$(find ros2_control_demo_description)/diffbot/urdf/diffbot_description.urdf.xacro" />
   <!-- Import Rviz colors -->
@@ -11,4 +12,12 @@
   <xacro:diffbot prefix="$(arg prefix)" />
   <xacro:diffbot_ros2_control
-    name="DiffBot" prefix="$(arg prefix)" use_mock_hardware="$(arg use_mock_hardware)"/>
+    name="DiffBot"
+    prefix="$(arg prefix)"
+    use_mock_hardware="$(arg use_mock_hardware)"
+    use_gazebo_classic="$(arg use_gazebo_classic)"/>
+  <xacro:if value="$(arg use_gazebo_classic)">
+    <!-- Import Gazebo Classic definitions + plugin -->
+    <xacro:include filename="$(find vmxpi_ros2)/gazebo/diffbot.gazebo.xacro" />
+    <xacro:diffbot_gazebo prefix="$(arg prefix)"/>
+  </xacro:if>
 </robot>

Commit message: adding TitanSystemHardware

File: description/ros2_control/diffbot.ros2_control.xacro (robot description, xacro)
@@ -1,7 +1,7 @@
 <?xml version="1.0"?>
 <robot xmlns:xacro="http://www.ros.org/wiki/xacro">
-  <xacro:macro name="diffbot_ros2_control" params="name prefix use_mock_hardware use_gazebo_classic">
+  <xacro:macro name="diffbot_ros2_control" params="name prefix use_hardware use_gazebo_classic">
     <ros2_control name="${name}" type="system">
-      <xacro:unless value="${use_mock_hardware}">
+      <xacro:unless value="${use_hardware}">
         <hardware>
           <plugin>vmxpi_ros2/DiffBotSystemHardware</plugin>
@@ -10,8 +10,7 @@
         </hardware>
       </xacro:unless>
-      <xacro:if value="${use_mock_hardware}">
+      <xacro:if value="${use_hardware}">
         <hardware>
-          <plugin>mock_components/GenericSystem</plugin>
-          <param name="calculate_dynamics">true</param>
+          <plugin>vmxpi_ros2/TitanSystemHardware</plugin>
         </hardware>
       </xacro:if>

File: description/urdf/diffbot.urdf.xacro (robot description, xacro)
@@ -3,5 +3,5 @@
 <robot xmlns:xacro="http://www.ros.org/wiki/xacro" name="diffdrive_robot">
   <xacro:arg name="prefix" default="" />
-  <xacro:arg name="use_mock_hardware" default="false" />
+  <xacro:arg name="use_hardware" default="false" />
   <xacro:arg name="use_gazebo_classic" default="false" />
   <xacro:include filename="$(find vmxpi_ros2)/diffbot/urdf/diffbot_description.urdf.xacro" />
@@ -14,5 +14,5 @@
     name="DiffBot"
     prefix="$(arg prefix)"
-    use_mock_hardware="$(arg use_mock_hardware)"
+    use_hardware="$(arg use_hardware)"
     use_gazebo_classic="$(arg use_gazebo_classic)"/>
   <xacro:if value="$(arg use_gazebo_classic)">
