Commit message: fix  diffbot with gazebo

File: description/diffbot/urdf/diffbot_description.urdf.xacro (robot description, xacro)
@@ -5,12 +5,12 @@
   <xacro:property name="PI" value="3.1415926535897931"/>
   <xacro:property name="base_mass" value="10.0" /> <!-- arbitrary value for base mass -->
-  <xacro:property name="base_width" value="0.2" />
-  <xacro:property name="base_length" value="0.2" />
+  <xacro:property name="base_width" value="0.4" />
+  <xacro:property name="base_length" value="0.4" />
   <xacro:property name="base_height" value="0.1" />
   <xacro:property name="wheel_mass" value="0.3" /> <!-- arbitrary value for wheel mass -->
   <xacro:property name="wheel_len" value="0.020" />
-  <xacro:property name="wheel_radius" value="0.015" />
+  <xacro:property name="wheel_radius" value="0.05" />
   <xacro:property name="caster_wheel_mass" value="0.1" /> <!-- arbitrary value for caster wheel mass -->
-  <xacro:property name="caster_wheel_radius" value="0.015" />
+  <xacro:property name="caster_wheel_radius" value="0.05" />
   <xacro:property name="z_offset" value="-${base_height/2}" /> <!-- Space btw top of beam and the each joint -->
   <!-- Base Link -->
@@ -41,5 +41,5 @@
       <parent link="${prefix}base_link"/>
       <child link="${prefix}left_wheel"/>
-      <origin xyz="0 -${base_width/2} ${z_offset}" rpy="0 0 0"/>
+      <origin xyz="0 ${base_width/2} ${z_offset}" rpy="0 0 0"/>
       <axis xyz="0 1 0"/>
       <dynamics damping="0.05"/>
@@ -73,5 +73,5 @@
       <parent link="${prefix}base_link"/>
       <child link="${prefix}right_wheel"/>
-      <origin xyz="0 ${base_width/2} ${z_offset}" rpy="0 0 0"/>
+      <origin xyz="0 -${base_width/2} ${z_offset}" rpy="0 0 0"/>
       <axis xyz="0 1 0"/>
       <dynamics damping="0.05"/>
@@ -120,5 +120,5 @@
           <sphere radius="${caster_wheel_radius}"/>
         </geometry>
-        <material name="white"/>
+        <material name="green"/>
       </visual>
       <inertial>

File: description/gazebo/diffbot.gazebo.xacro (robot description, xacro)
@@ -14,7 +14,6 @@
     <!-- Joint State Publisher Plugin -->
     <gazebo>
-      <plugin name="gazebo_ros_joint_state_publisher" filename="libgazebo_ros_joint_state_publisher.so">
-        <update_rate>50</update_rate>  <!-- Adjust the rate as needed -->
-        <!-- <joint_prefix>${prefix}</joint_prefix>  Ensures proper naming -->
+      <plugin name="gazebo_joint_state_broadcaster" filename="libgazebo_ros_joint_state_publisher.so">
+        <update_rate>10</update_rate>  <!-- Adjust the rate as needed -->
         <joint_name>${prefix}right_wheel_joint</joint_name>
         <joint_name>${prefix}left_wheel_joint</joint_name>
@@ -29,6 +28,6 @@
     <!-- Left Wheel -->
     <gazebo reference="${prefix}left_wheel">
-      <kp>1000000.0</kp>
-      <kd>10.0</kd>
+      <kp>1e6</kp>
+      <kd>1e4</kd>
       <friction>
         <ode>
@@ -41,6 +40,6 @@
     <!-- Right Wheel -->
     <gazebo reference="${prefix}right_wheel">
-      <kp>1000000.0</kp>
-      <kd>10.0</kd>
+      <kp>1e6</kp>
+      <kd>1e4</kd>
       <friction>
         <ode>
@@ -53,6 +52,6 @@
     <!-- Caster Frontal Wheel -->
     <gazebo reference="${prefix}caster_frontal_wheel">
-      <kp>1000000.0</kp>  <!-- Lower than drive wheels -->
-      <kd>5.0</kd>
+      <kp>1e6</kp>
+      <kd>1e4</kd>
       <friction>
         <ode>
@@ -61,10 +60,10 @@
         </ode>
       </friction>
-      <material>Gazebo/White</material>
+      <material>Gazebo/Green</material>
     </gazebo>
     <!-- Caster Rear Wheel -->
     <gazebo reference="${prefix}caster_rear_wheel">
-      <kp>1000000.0</kp>
-      <kd>5.0</kd>
+      <kp>1e6</kp>
+      <kd>1e4</kd>
       <friction>
         <ode>

Commit message: working

File: description/diffbot/urdf/diffbot_description.urdf.xacro (robot description, xacro)
@@ -14,6 +14,8 @@
   <xacro:property name="caster_wheel_radius" value="0.05" />
   <xacro:property name="z_offset" value="-${base_height/2}" /> <!-- Space btw top of beam and the each joint -->
+  <link name="${prefix}base_link">
+  </link>
   <!-- Base Link -->
-  <link name="${prefix}base_link">
+  <link name="${prefix}chassis_link">
     <collision>
       <origin xyz="0 0 0" rpy="0 0 0"/>
@@ -38,6 +40,11 @@
       </inertial>
     </link>
+    <joint name="${prefix}base_link_joint" type="fixed">
+      <origin rpy="0 0 0" xyz="0 0 0" />
+      <parent link="${prefix}base_link" />
+      <child link="${prefix}chassis_link" />
+    </joint>
     <joint name="${prefix}left_wheel_joint" type="continuous">
-      <parent link="${prefix}base_link"/>
+      <parent link="${prefix}chassis_link"/>
       <child link="${prefix}left_wheel"/>
       <origin xyz="0 ${base_width/2} ${z_offset}" rpy="0 0 0"/>
@@ -71,5 +78,5 @@
       </link>
     <joint name="${prefix}right_wheel_joint" type="continuous">
-      <parent link="${prefix}base_link"/>
+      <parent link="${prefix}chassis_link"/>
       <child link="${prefix}right_wheel"/>
       <origin xyz="0 -${base_width/2} ${z_offset}" rpy="0 0 0"/>
@@ -103,5 +110,5 @@
       </link>
     <joint name="${prefix}caster_frontal_wheel_joint" type="continuous">
-      <parent link="${prefix}base_link"/>
+      <parent link="${prefix}chassis_link"/>
       <child link="${prefix}caster_frontal_wheel"/>
       <origin xyz="${base_width/2 - caster_wheel_radius} 0 ${z_offset}" rpy="0 0 0"/>
@@ -132,5 +139,5 @@
       </link>
     <joint name="${prefix}caster_rear_wheel_joint" type="continuous">
-      <parent link="${prefix}base_link"/>
+      <parent link="${prefix}chassis_link"/>
       <child link="${prefix}caster_rear_wheel"/>
       <origin xyz="${-base_width/2 + caster_wheel_radius} 0 ${z_offset}" rpy="0 0 0"/>
@@ -160,4 +167,37 @@
         </inertial>
       </link>
+      <!-- <link name="${prefix}laser_model_link">
+        <visual>
+          <origin rpy="0 0 0" xyz="0 0 0"/>
+          <geometry>
+            <mesh filename="package://vmxpi_ros2/meshes/sensors/hokuyo_urg_04lx.dae" scale="1.0 1.0 1.0"/>
+          </geometry>
+        </visual>
+        <collision>
+          <origin rpy="0 0 0" xyz="0 0 0"/>
+          <geometry>
+            <mesh filename="package://vmxpi_ros2/meshes/sensors/hokuyo_urg_04lx.dae" scale="1.0 1.0 1.0"/>
+          </geometry>
+        </collision>
+        <inertial>
+          <mass value="0.01"/>
+          <origin rpy="0 0 0" xyz="0 0 0"/>
+          <inertia ixx="6.066578520833334e-06" ixy="0" ixz="0" iyy="6.072950163333333e-06" iyz="0" izz="9.365128684166666e-06"/>
+        </inertial>
+      </link>
+      <joint name="${prefix}laser_scan_model_link_joint" type="fixed">
+        <origin rpy="0 0 0" xyz="0.0 0.0 ${base_height}"/>
+        <parent link="${prefix}chassis_link"/>
+        <child link="${prefix}laser_model_link"/>
+        <axis xyz="0 0 0"/>
+      </joint>
+      <link name="${prefix}laser_scan_frame">
+        <origin rpy="0 0 0" xyz="0 0 ${base_height}"/>
+      </link>
+      <joint name="${prefix}laser_scan_frame_joint" type="fixed">
+        <origin rpy="0 0 0" xyz="0 0 0.05"/>
+        <parent link="${prefix}laser_model_link"/>
+        <child link="${prefix}laser_scan_frame"/>
+      </joint> -->
   </xacro:macro>
 </robot>

File: description/gazebo/diffbot.gazebo.xacro (robot description, xacro)
@@ -16,12 +16,15 @@
       <plugin name="gazebo_joint_state_broadcaster" filename="libgazebo_ros_joint_state_publisher.so">
         <update_rate>10</update_rate>  <!-- Adjust the rate as needed -->
-        <joint_name>${prefix}right_wheel_joint</joint_name>
-        <joint_name>${prefix}left_wheel_joint</joint_name>
+        <!-- <joint_name>${prefix}base_link_joint</joint_name> -->
+        <!-- <joint_name>${prefix}right_wheel_joint</joint_name> -->
+        <!-- <joint_name>${prefix}left_wheel_joint</joint_name> -->
         <joint_name>${prefix}caster_frontal_wheel_joint</joint_name>
         <joint_name>${prefix}caster_rear_wheel_joint</joint_name>
+        <!-- <joint_name>${prefix}laser_scan_frame_joint</joint_name>
+        <joint_name>${prefix}laser_scan_model_link_joint</joint_name>    -->
       </plugin>
     </gazebo>
     <!-- Base Link -->
-    <gazebo reference="${prefix}base_link">
+    <gazebo reference="${prefix}chassis_link">
       <material>Gazebo/Orange</material>
     </gazebo>
@@ -74,4 +77,33 @@
       <material>Gazebo/White</material>
     </gazebo>
+    <!-- <gazebo reference="${prefix}laser_scan_frame">
+      <sensor name="sensor_ray" type="ray">
+          <pose>0 0 0 0 0 0</pose>
+          <ray>
+            <scan>
+              <horizontal>
+                <samples>200</samples>
+                <resolution>1.0</resolution>
+                <min_angle>-3.14</min_angle>
+                <max_angle>3.14</max_angle>
+              </horizontal>
+            </scan>
+            <range>
+              <min>0.1</min>
+              <max>5.0</max>
+            </range>
+          </ray>
+          <always_on>true</always_on>
+          <visualize>true</visualize>
+          <update_rate>100.0</update_rate>
+          <plugin name="laser_scan_node" filename="libgazebo_ros_ray_sensor.so">
+            <ros>
+              <remapping>~/out:=scan</remapping>
+            </ros>
+            <frame_name>${prefix}laser_scan_frame</frame_name>
+            <output_type>sensor_msgs/LaserScan</output_type>
+          </plugin>
+      </sensor>
+    </gazebo> -->
   </xacro:macro>
 </robot>

Commit message: laser is working in gazevo and rviz

File: description/diffbot/urdf/diffbot_description.urdf.xacro (robot description, xacro)
@@ -167,9 +167,10 @@
         </inertial>
       </link>
-      <!-- <link name="${prefix}laser_model_link">
+      <link name="${prefix}laser_model_link">
         <visual>
           <origin rpy="0 0 0" xyz="0 0 0"/>
           <geometry>
-            <mesh filename="package://vmxpi_ros2/meshes/sensors/hokuyo_urg_04lx.dae" scale="1.0 1.0 1.0"/>
+            <!-- <mesh filename="package://vmxpi_ros2/description/meshes/sensors/hokuyo_urg_04lx.dae" scale="1.0 1.0 1.0"/> -->
+            <cylinder length="0.05" radius="0.05"/>
           </geometry>
         </visual>
@@ -177,5 +178,6 @@
           <origin rpy="0 0 0" xyz="0 0 0"/>
           <geometry>
-            <mesh filename="package://vmxpi_ros2/meshes/sensors/hokuyo_urg_04lx.dae" scale="1.0 1.0 1.0"/>
+            <!-- <mesh filename="package://vmxpi_ros2/description/meshes/sensors/hokuyo_urg_04lx.dae" scale="1.0 1.0 1.0"/> -->
+            <cylinder length="0.05" radius="0.05"/>
           </geometry>
         </collision>
@@ -199,5 +201,5 @@
         <parent link="${prefix}laser_model_link"/>
         <child link="${prefix}laser_scan_frame"/>
-      </joint> -->
+      </joint>
   </xacro:macro>
 </robot>

File: description/gazebo/diffbot.gazebo.xacro (robot description, xacro)
@@ -77,5 +77,5 @@
       <material>Gazebo/White</material>
     </gazebo>
-    <!-- <gazebo reference="${prefix}laser_scan_frame">
+    <gazebo reference="${prefix}laser_scan_frame">
       <sensor name="sensor_ray" type="ray">
           <pose>0 0 0 0 0 0</pose>
@@ -105,5 +105,5 @@
           </plugin>
       </sensor>
-    </gazebo> -->
+    </gazebo>
   </xacro:macro>
 </robot>

Commit message: laser is working with sim

File: description/diffbot/urdf/diffbot_description.urdf.xacro (robot description, xacro)
@@ -171,6 +171,6 @@
           <origin rpy="0 0 0" xyz="0 0 0"/>
           <geometry>
-            <!-- <mesh filename="package://vmxpi_ros2/description/meshes/sensors/hokuyo_urg_04lx.dae" scale="1.0 1.0 1.0"/> -->
-            <cylinder length="0.05" radius="0.05"/>
+            <!-- <mesh filename="package://vmxpi_ros2/meshes/sensors/hokuyo_urg_04lx.dae" scale="1.0 1.0 1.0"/> -->
+            <cylinder length="0.1" radius="0.05"/>
           </geometry>
         </visual>
@@ -178,6 +178,6 @@
           <origin rpy="0 0 0" xyz="0 0 0"/>
           <geometry>
-            <!-- <mesh filename="package://vmxpi_ros2/description/meshes/sensors/hokuyo_urg_04lx.dae" scale="1.0 1.0 1.0"/> -->
-            <cylinder length="0.05" radius="0.05"/>
+            <!-- <mesh filename="package://vmxpi_ros2/meshes/sensors/hokuyo_urg_04lx.dae" scale="1.0 1.0 1.0"/> -->
+            <cylinder length="0.1" radius="0.05"/>
           </geometry>
         </collision>

Commit message: working in rviz but  mesh file not loading in Gazebo

File: description/diffbot/urdf/diffbot_description.urdf.xacro (robot description, xacro)
@@ -171,6 +171,6 @@
           <origin rpy="0 0 0" xyz="0 0 0"/>
           <geometry>
-            <!-- <mesh filename="package://vmxpi_ros2/meshes/sensors/hokuyo_urg_04lx.dae" scale="1.0 1.0 1.0"/> -->
-            <cylinder length="0.1" radius="0.05"/>
+            <mesh filename="package://vmxpi_ros2/meshes/sensors/hokuyo_urg_04lx.dae" scale="1.0 1.0 1.0"/>
+            <!-- <cylinder length="0.1" radius="0.05"/> -->
           </geometry>
         </visual>
@@ -178,6 +178,6 @@
           <origin rpy="0 0 0" xyz="0 0 0"/>
           <geometry>
-            <!-- <mesh filename="package://vmxpi_ros2/meshes/sensors/hokuyo_urg_04lx.dae" scale="1.0 1.0 1.0"/> -->
-            <cylinder length="0.1" radius="0.05"/>
+            <mesh filename="package://vmxpi_ros2/meshes/sensors/hokuyo_urg_04lx.dae" scale="1.0 1.0 1.0"/>
+            <!-- <cylinder length="0.1" radius="0.05"/> -->
           </geometry>
         </collision>

File: description/gazebo/diffbot.gazebo.xacro (robot description, xacro)
@@ -15,5 +15,5 @@
     <gazebo>
       <plugin name="gazebo_joint_state_broadcaster" filename="libgazebo_ros_joint_state_publisher.so">
-        <update_rate>10</update_rate>  <!-- Adjust the rate as needed -->
+        <update_rate>100</update_rate>  <!-- Adjust the rate as needed -->
         <!-- <joint_name>${prefix}base_link_joint</joint_name> -->
         <!-- <joint_name>${prefix}right_wheel_joint</joint_name> -->

Commit message: fixing gazebo issue

File: description/diffbot/urdf/diffbot_description.urdf.xacro (robot description, xacro)
@@ -171,5 +171,5 @@
           <origin rpy="0 0 0" xyz="0 0 0"/>
           <geometry>
-            <mesh filename="package://vmxpi_ros2/meshes/sensors/hokuyo_urg_04lx.dae" scale="1.0 1.0 1.0"/>
+            <mesh filename="package://vmxpi_ros2/description/meshes/sensors/hokuyo_urg_04lx.dae" scale="1.0 1.0 1.0"/>
             <!-- <cylinder length="0.1" radius="0.05"/> -->
           </geometry>
@@ -178,5 +178,5 @@
           <origin rpy="0 0 0" xyz="0 0 0"/>
           <geometry>
-            <mesh filename="package://vmxpi_ros2/meshes/sensors/hokuyo_urg_04lx.dae" scale="1.0 1.0 1.0"/>
+            <mesh filename="package://vmxpi_ros2/description/meshes/sensors/hokuyo_urg_04lx.dae" scale="1.0 1.0 1.0"/>
             <!-- <cylinder length="0.1" radius="0.05"/> -->
           </geometry>

File: description/urdf/diffbot.urdf.xacro (robot description, xacro)
@@ -5,9 +5,9 @@
   <xacro:arg name="use_hardware" default="false" />
   <xacro:arg name="use_gazebo_classic" default="false" />
-  <xacro:include filename="$(find vmxpi_ros2)/diffbot/urdf/diffbot_description.urdf.xacro" />
+  <xacro:include filename="$(find vmxpi_ros2)/description/diffbot/urdf/diffbot_description.urdf.xacro" />
   <!-- Import Rviz colors -->
-  <xacro:include filename="$(find vmxpi_ros2)/diffbot/urdf/diffbot.materials.xacro" />
+  <xacro:include filename="$(find vmxpi_ros2)/description/diffbot/urdf/diffbot.materials.xacro" />
   <!-- Import diffbot ros2_control description -->
-  <xacro:include filename="$(find vmxpi_ros2)/ros2_control/diffbot.ros2_control.xacro" />
+  <xacro:include filename="$(find vmxpi_ros2)/description/ros2_control/diffbot.ros2_control.xacro" />
   <xacro:diffbot prefix="$(arg prefix)" />
   <xacro:diffbot_ros2_control
@@ -18,5 +18,5 @@
   <xacro:if value="$(arg use_gazebo_classic)">
     <!-- Import Gazebo Classic definitions + plugin -->
-    <xacro:include filename="$(find vmxpi_ros2)/gazebo/diffbot.gazebo.xacro" />
+    <xacro:include filename="$(find vmxpi_ros2)/description/gazebo/diffbot.gazebo.xacro" />
     <xacro:diffbot_gazebo prefix="$(arg prefix)"/>
   </xacro:if>

Commit message: working in VMX

File: description/diffbot/urdf/diffbot_description.urdf.xacro (robot description, xacro)
@@ -9,5 +9,5 @@
   <xacro:property name="base_height" value="0.1" />
   <xacro:property name="wheel_mass" value="0.3" /> <!-- arbitrary value for wheel mass -->
-  <xacro:property name="wheel_len" value="0.020" />
+  <xacro:property name="wheel_len" value="0.04" />
   <xacro:property name="wheel_radius" value="0.05" />
   <xacro:property name="caster_wheel_mass" value="0.1" /> <!-- arbitrary value for caster wheel mass -->

File: description/gazebo/diffbot.gazebo.xacro (robot description, xacro)
@@ -15,5 +15,5 @@
     <gazebo>
       <plugin name="gazebo_joint_state_broadcaster" filename="libgazebo_ros_joint_state_publisher.so">
-        <update_rate>100</update_rate>  <!-- Adjust the rate as needed -->
+        <update_rate>50</update_rate>  <!-- Adjust the rate as needed -->
         <!-- <joint_name>${prefix}base_link_joint</joint_name> -->
         <!-- <joint_name>${prefix}right_wheel_joint</joint_name> -->
